File: neptune-camera-esp/neptune-camera-esp.kicad_pcb (KiCad board)
At the start: 4 copper layers, 50 x 50 mm, 40 parts, among them J1 Conn_02x10_Odd_Even, J2 Conn_02x10_Odd_Even, J3 ov5640, SW1 EN_Button, SW2 BOOT_Button, U1 ESP32-S3-WROOM-1, U2 TLV74315, U3 TLV74328, U4 AP2112K-3.3, Y1 ECS-2520MVQ-240-BS-TR

Commit message: -
Parts:
- added J5: Programmersocket, neptune-camera-esp-footprints:PinSocket_1x05_P2.54mm_Horizontal, B.Cu at (117.7, 49.9)
- added R5: 10k, Resistor_SMD:R_0402_1005Metric, F.Cu at (113.2, 55.1)
- added R6: 10k, Resistor_SMD:R_0402_1005Metric, F.Cu at (113.2, 57.4)
Connections:
- J1 pad 3: /I2C_OBC_SDA -> /I2C_OBC_SCL
- J3 pad 9: /HYSNC -> /HSYNC
- U1 pad 15: unconnected-(U1-IO3-Pad15) -> /D4
- U1 pad 16: unconnected-(U1-IO46-Pad16) -> /D3
- U1 pad 17: unconnected-(U1-IO9-Pad17) -> /D5
- U1 pad 18: unconnected-(U1-IO10-Pad18) -> /D2
- U1 pad 19: unconnected-(U1-IO11-Pad19) -> /D6
- U1 pad 20: unconnected-(U1-IO12-Pad20) -> /PCLK
- U1 pad 21: unconnected-(U1-IO13-Pad21) -> /D7
- U1 pad 22: unconnected-(U1-IO14-Pad22) -> /D8
- U1 pad 23: unconnected-(U1-IO21-Pad23) -> /D9
- U1 pad 24: unconnected-(U1-IO47-Pad24) -> /HSYNC
- U1 pad 25: unconnected-(U1-IO48-Pad25) -> /VSYNC
- U1 pad 31: unconnected-(U1-IO38-Pad31) -> /OV5640_SCL
- U1 pad 32: unconnected-(U1-IO39-Pad32) -> /OV5640_SDA
- U1 pad 36: unconnected-(U1-RXD0-Pad36) -> /PRG_UART_RX
- U1 pad 37: unconnected-(U1-TXD0-Pad37) -> /PRG_UART_TX
- U1 pad 7: unconnected-(U1-IO7-Pad7) -> /I2C_OBC_SDA
- U1 pad 8: unconnected-(U1-IO15-Pad8) -> /I2C_OBC_SCL
Routing:
- net /BOOT: track 0.00 -> 34.3 mm, vias 0 -> 2
- net /OV5640_SDA: track 0.00 -> 31.7 mm, vias 0 -> 1
- net /OV5640_SCL: track 0.00 -> 30.2 mm, vias 0 -> 1
- net /HSYNC: track 0.00 -> 19.9 mm, vias 0 -> 1
- net /VSYNC: track 0.00 -> 19.7 mm, vias 0 -> 1
- net /D8: track 0.00 -> 19.5 mm, vias 0 -> 1
- net /D9: track 0.00 -> 19.4 mm, vias 0 -> 1
- net /D7: track 0.00 -> 19.2 mm, vias 0 -> 1
- net /D4: track 0.00 -> 19.1 mm, vias 0 -> 1
- net /PCLK: track 1.48 -> 20.4 mm, vias 0 -> 1
- net /D3: track 0.00 -> 18.8 mm, vias 0 -> 1
- net /D6: track 0.00 -> 18.6 mm, vias 0 -> 1
- net /D5: track 0.00 -> 18.5 mm, vias 0 -> 1
- net /D2: track 0.00 -> 18.2 mm, vias 0 -> 1
- net VCC: track 28.6 -> 44.1 mm, vias 0 -> 1
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Other:
- board text added: "AF"

Commit message: Production
Connections:
- U1 pad 34: unconnected-(U1-IO41-Pad34) -> /LTE_PWRKEY
- U1 pad 35: unconnected-(U1-IO42-Pad35) -> /LTE_RESET
Routing:
- net /LTE_RESET: track 0.00 -> 21.6 mm
- net /LTE_PWRKEY: track 0.00 -> 16.9 mm
- net VCC: track 44.1 -> 39.6 mm, vias 1 -> 2
Other:
- board text added: "Camera Module"
- board text added: "revision 1.0-b Project Neptune"
