File: neptune-camera-esp/neptune-camera-esp.kicad_pcb (KiCad board)
At the start: 4 copper layers, 50 x 50 mm, 43 parts, among them J1 Conn_02x10_Odd_Even, J2 Conn_02x10_Odd_Even, J3 ov5640, J5 Programmersocket, SW1 EN_Button, SW2 BOOT_Button, U1 ESP32-S3-WROOM-1, U2 TLV74315, U3 TLV74328, U4 AP2112K-3.3, Y1 ECS-2520MVQ-240-BS-TR

Commit message: kondi érték hiba javitasa
Parts:
- C22: value 22uF -> 100nF

Commit message: megyek ebédelni :)
Parts:
- removed C20: 22pF, Capacitor_SMD:C_0402_1005Metric
- removed Y1: ECS-2520MVQ-240-BS-TR, neptune-camera-esp-footprints:ECS2520MVQ240BSTR
- added R10: 22, Resistor_SMD:R_0402_1005Metric, B.Cu at (92.1, 46.7)
- added R7: 22, Resistor_SMD:R_0402_1005Metric, B.Cu at (92.1, 50.5)
- added R8: 22, Resistor_SMD:R_0402_1005Metric, B.Cu at (92.1, 49.3)
- added R9: 22, Resistor_SMD:R_0402_1005Metric, B.Cu at (92.1, 48.0)
- C22, C23: moved to B.Cu
- C25: moved to F.Cu
- U1: footprint neptune-camera-esp-footprints:ESP32-S3-WROOM-1 -> neptune-camera-esp-footprints:ESP32-S3-WROOM-1U; moved to B.Cu
- moved R5 39.6 mm to (142.2, 82.1)
- moved R6 38.8 mm to (143.4, 81.7)
- moved C21 28.8 mm to (134.4, 79.9)
- moved R2 27.8 mm to (132.9, 80.0)
- moved R1 27.5 mm to (133.0, 78.3)
- moved C23 25.5 mm to (115.2, 39.8)
- moved C22 22.0 mm to (113.4, 39.8)
- moved R3 6.25 mm to (88.3, 44.0), turned to 180 degrees
- moved C24 5.59 mm to (88.3, 43.0), turned to 0 degrees
- moved C25 3.23 mm to (84.2, 43.1)
- moved U1 3.18 mm to (102.9, 47.5), turned to 180 degrees
- moved R4 1.02 mm to (87.8, 45.5), turned to 90 degrees
Connections:
- R5 pad 1: /OV5640_SDA -> unconnected-(R5-Pad1)
- R5 pad 2: +3.3V -> unconnected-(R5-Pad2)
- R6 pad 1: +3.3V -> unconnected-(R6-Pad1)
- R6 pad 2: /OV5640_SCL -> unconnected-(R6-Pad2)
- U1 pad 15: /D4 -> unconnected-(U1-IO3-Pad15)
- U1 pad 16: /D3 -> unconnected-(U1-IO46-Pad16)
- U1 pad 17: /D5 -> unconnected-(U1-IO9-Pad17)
- U1 pad 18: /D2 -> unconnected-(U1-IO10-Pad18)
- U1 pad 19: /D6 -> unconnected-(U1-IO11-Pad19)
- U1 pad 20: /PCLK -> unconnected-(U1-IO12-Pad20)
- U1 pad 21: /D7 -> unconnected-(U1-IO13-Pad21)
- U1 pad 22: /D8 -> unconnected-(U1-IO14-Pad22)
- U1 pad 23: /D9 -> unconnected-(U1-IO21-Pad23)
- U1 pad 24: /HSYNC -> unconnected-(U1-IO47-Pad24)
- U1 pad 25: /VSYNC -> unconnected-(U1-IO48-Pad25)
- U1 pad 31: /OV5640_SCL -> Net-(U1-IO38)
- U1 pad 32: /OV5640_SDA -> Net-(U1-IO39)
- U1 pad 33: unconnected-(U1-IO40-Pad33) -> Net-(U1-IO40)
- U1 pad 34: /LTE_PWRKEY -> Net-(U1-IO41)
- U1 pad 35: /LTE_RESET -> unconnected-(U1-IO42-Pad35)
- U1 pad 7: /I2C_OBC_SDA -> unconnected-(U1-IO7-Pad7)
- U1 pad 8: /I2C_OBC_SCL -> unconnected-(U1-IO15-Pad8)
Routing:
- net /OV5640_SDA: track 31.7 -> 0.00 mm, vias 1 -> 0
- net /OV5640_SCL: track 30.2 -> 0.00 mm, vias 1 -> 0
- net GND: track 88.9 -> 62.8 mm, vias 30 -> 19
- net /BOOT: track 34.3 -> 10.1 mm, vias 2 -> 1
- net /LTE_RESET: track 21.6 -> 0.00 mm
- net /PCLK: track 20.4 -> 0.00 mm, vias 1 -> 0
- net /HSYNC: track 19.9 -> 0.00 mm, vias 1 -> 0
- net /D4: track 19.1 -> 39.0 mm, vias 1 -> 0
- net /VSYNC: track 19.7 -> 0.00 mm, vias 1 -> 0
- net /D8: track 19.5 -> 0.00 mm, vias 1 -> 0
- net /D9: track 19.4 -> 0.00 mm, vias 1 -> 0
- net /D7: track 19.2 -> 0.00 mm, vias 1 -> 0
- net /D3: track 18.8 -> 37.4 mm, vias 1 -> 0
- net /D6: track 18.6 -> 0.00 mm, vias 1 -> 0
- net /D5: track 18.5 -> 35.8 mm, vias 1 -> 0
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- removed copper zone on In2.Cu, net +3.3V
- removed copper zone on In1.Cu, net GND

Commit message: finom volt az ebéd, megyek haza
Parts:
- removed R10, R7, R8, R9: 22, Resistor_SMD:R_0402_1005Metric
Connections:
- C21 pad 1: /Camera(OV5640)/CameraReset -> /CAM_PWDN
- J3 pad 13: /Camera(OV5640)/XCLK -> /PCLK
- J3 pad 6: /Camera(OV5640)/CameraReset -> /CAM_PWDN
- J3 pad 8: /Camera(OV5640)/CameraPWDN -> /CAM_RESET
- R1 pad 1: /Camera(OV5640)/CameraReset -> /CAM_PWDN
- R2 pad 1: /Camera(OV5640)/CameraPWDN -> /CAM_RESET
- R5 pad 1: unconnected-(R5-Pad1) -> +3.3V
- R5 pad 2: unconnected-(R5-Pad2) -> /OV5640_SDA
- R6 pad 1: unconnected-(R6-Pad1) -> /OV5640_SCL
- R6 pad 2: unconnected-(R6-Pad2) -> +3.3V
- U1 pad 12: unconnected-(U1-IO8-Pad12) -> /OV5640_SCL
- U1 pad 17: unconnected-(U1-IO9-Pad17) -> /CAM_PWDN
- U1 pad 18: unconnected-(U1-IO10-Pad18) -> /VSYNC
- U1 pad 19: unconnected-(U1-IO11-Pad19) -> /CAM_RESET
- U1 pad 20: unconnected-(U1-IO12-Pad20) -> /HSYNC
- U1 pad 21: unconnected-(U1-IO13-Pad21) -> /D9
- U1 pad 22: unconnected-(U1-IO14-Pad22) -> /PCLK
- U1 pad 23: unconnected-(U1-IO21-Pad23) -> /D8
- U1 pad 24: unconnected-(U1-IO47-Pad24) -> /D7
- U1 pad 25: unconnected-(U1-IO48-Pad25) -> /PCLK
- U1 pad 26: unconnected-(U1-IO45-Pad26) -> /D6
- U1 pad 31: Net-(U1-IO38) -> /D2
- U1 pad 32: Net-(U1-IO39) -> /D5
- U1 pad 33: Net-(U1-IO40) -> /D3
- U1 pad 34: Net-(U1-IO41) -> /D4
- U1 pad 7: unconnected-(U1-IO7-Pad7) -> /OV5640_SDA
Routing:
- net Net-(U1-IO41): track 1.49 -> 0.00 mm
- net Net-(U1-IO40): track 1.49 -> 0.00 mm
- net Net-(U1-IO39): track 1.49 -> 0.00 mm
- net Net-(U1-IO38): track 1.49 -> 0.00 mm
- net /D2: track 34.2 -> 35.6 mm
- net /D5: track 35.8 -> 37.0 mm
- net /D3: track 37.4 -> 38.4 mm
- net /D4: track 39.0 -> 39.8 mm

Commit message: már nincs sok :)
Parts:
- added C20: 1uF, Capacitor_SMD:C_0603_1608Metric, F.Cu at (121.4, 50.5)
- added C26: 1uF, Capacitor_SMD:C_0603_1608Metric, F.Cu at (121.9, 44.7)
- added U5: AP2112K-3.3, neptune-camera-esp-footprints:SOT-23-5, F.Cu at (121.9, 47.6)
- moved C21 11.9 mm to (145.8, 76.7), turned to 0 degrees
- moved R2 10.1 mm to (142.9, 78.7), turned to 0 degrees
- moved R1 10.0 mm to (142.9, 76.7), turned to 0 degrees
- moved C10 5.88 mm to (119.2, 75.4), turned to 90 degrees
- moved C9 3.92 mm to (125.0, 75.9), turned to -90 degrees
- moved U4 3.17 mm to (122.1, 75.4), turned to 180 degrees
- moved R6 2.96 mm to (142.9, 84.6), turned to 0 degrees
- moved R5 0.91 mm to (142.9, 82.6), turned to 0 degrees
Connections:
- C22 pad 2: +3.3V -> +3.3VA
- C23 pad 2: +3.3V -> +3.3VA
- J3 pad 13: /PCLK -> /XCLK
- R3 pad 1: +3.3V -> +3.3VA
- R5 pad 1: +3.3V -> +3.3VA
- R6 pad 2: +3.3V -> +3.3VA
- U1 pad 10: unconnected-(U1-IO17-Pad10) -> /LTE_PWRKEY
- U1 pad 12: /OV5640_SCL -> unconnected-(U1-IO8-Pad12)
- U1 pad 15: unconnected-(U1-IO3-Pad15) -> /OV5640_SDA
- U1 pad 16: unconnected-(U1-IO46-Pad16) -> /OV5640_SCL
- U1 pad 2: +3.3V -> +3.3VA
- U1 pad 22: /PCLK -> /XCLK
- U1 pad 38: unconnected-(U1-IO2-Pad38) -> /I2C_OBC_SCL
- U1 pad 39: unconnected-(U1-IO1-Pad39) -> /I2C_OBC_SDA
- U1 pad 7: /OV5640_SDA -> unconnected-(U1-IO7-Pad7)
- U1 pad 9: unconnected-(U1-IO16-Pad9) -> /LTE_RESET
Routing:
- net /USB_DN: track 0.00 -> 46.4 mm, vias 0 -> 1
- net /USB_DP: track 0.00 -> 46.2 mm, vias 0 -> 1
- net GND: track 62.8 -> 107.3 mm, vias 19 -> 34
- net +3.3VA: track 0.00 -> 42.2 mm, vias 0 -> 1
- net /PRG_UART_RX: track 0.00 -> 28.4 mm, vias 0 -> 2
- net /PRG_UART_TX: track 0.00 -> 28.3 mm, vias 0 -> 2
- net /EN: track 0.00 -> 27.8 mm, vias 0 -> 1
- net /D6: track 0.00 -> 26.3 mm
- net /PCLK: track 0.00 -> 26.0 mm
- net /D7: track 0.00 -> 25.6 mm
- net /D8: track 0.00 -> 25.5 mm
- net /OV5640_SDA: track 0.00 -> 25.5 mm
- net /OV5640_SCL: track 0.00 -> 25.3 mm
- net /XCLK: track 0.00 -> 25.2 mm
- net /CAM_PWDN: track 0.00 -> 25.0 mm
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Other:
- board text added: "GND"
- board text added: "RX"
- board text added: "TX"
- board text added: "VCC"
- board text added: "revision 1.1 Project Neptune"
- board text removed: "revision 1.0-b Project Neptune"

Commit message: menni kell a vonathoz
Parts:
- moved R6 45.6 mm to (108.6, 54.6), turned to 90 degrees
- moved R2 45.0 mm to (104.8, 54.6), turned to 90 degrees
- moved C21 44.5 mm to (106.9, 55.1), turned to 180 degrees
- moved R5 43.3 mm to (109.9, 54.6), turned to -90 degrees
- moved R1 42.5 mm to (106.8, 54.1), turned to 180 degrees
- moved JP1 1.24 mm to (97.0, 83.7)
Routing:
- net +3.3V: track 32.1 -> 70.8 mm, vias 3 -> 2
- net /CAM_PWDN: track 25.0 -> 27.8 mm, vias 0 -> 1
- net /OV5640_SDA: track 25.5 -> 27.2 mm, vias 0 -> 1
- net /OV5640_SCL: track 25.3 -> 27.1 mm, vias 0 -> 1
- net /CAM_RESET: track 24.7 -> 26.4 mm, vias 0 -> 1
- net GND: track 107.3 -> 108.6 mm, vias 34 -> 36
- net Net-(J3-AF-VCC): track 3.18 -> 2.26 mm

Commit message: még kellenek stiching viák, meg át kell nézni
Connections:
- R1 pad 2: +3.3V -> +3.3VA
Routing:
- net +3.3VA: track 42.2 -> 68.7 mm
- net +3.3V: track 70.8 -> 81.7 mm, vias 2 -> 3
- added copper zone on In1.Cu, net GND
- added copper zone on In2.Cu, net GND
Changed lines of the file:
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@@
 			(layers "F.Cu" "F.Mask" "F.Paste")
 			(roundrect_rratio 0.25)
-			(net "+3.3V")
+			(net "+3.3VA")
 			(pintype "passive")
 		)
@@
 	)
 	(segment
+		(start 106.323 54.109)
+		(end 106.323 52.658)
+		(width 0.5)
+		(layer "F.Cu")
+		(net "+3.3VA")
+	)
+	(segment
 		(start 91.289 44.001)
 		(end 94.579 40.711)
@@
 	)
 	(segment
+		(start 106.408 52.573)
+		(end 99.861 52.573)
+		(width 0.5)
+		(layer "F.Cu")
+		(net "+3.3VA")
+	)
+	(segment
+		(start 109.432 52.573)
+		(end 108.532 52.573)
+		(width 0.5)
+		(layer "F.Cu")
+		(net "+3.3VA")
+	)
+	(segment
+		(start 109.883 54.109)
+		(end 109.883 53.024)
+		(width 0.5)
+		(layer "F.Cu")
+		(net "+3.3VA")
+	)
+	(segment
+		(start 108.613 54.109)
+		(end 108.613 52.654)
+		(width 0.5)
+		(layer "F.Cu")
+		(net "+3.3VA")
+	)
+	(segment
 		(start 88.831 44.001)
 		(end 91.289 44.001)
@@
 	)
 	(segment
+		(start 109.883 53.024)
+		(end 109.432 52.573)
+		(width 0.5)
+		(layer "F.Cu")
+		(net "+3.3VA")
+	)
+	(segment
 		(start 120.9755 44.874)
 		(end 121.1505 44.699)
@@
 	)
 	(segment
+		(start 106.323 52.658)
+		(end 106.408 52.573)
+		(width 0.5)
+		(layer "F.Cu")
+		(net "+3.3VA")
+	)
+	(segment
 		(start 120.9755 46.4615)
 		(end 120.9755 44.874)
@@
 		(net "+3.3VA")
 	)
+	(segment
+		(start 99.861 52.573)
+		(end 91.289 44.001)
+		(width 0.5)
+		(layer "F.Cu")
+		(net "+3.3VA")
+	)
+	(segment
+		(start 108.613 52.654)
+		(end 108.532 52.573)
+		(width 0.5)
+		(layer "F.Cu")
+		(net "+3.3VA")
+	)
+	(segment
+		(start 108.532 52.573)
+		(end 106.408 52.573)
+		(width 0.5)
+		(layer "F.Cu")
+		(net "+3.3VA")
+	)
 	(via
 		(at 116.517 40.711)
@@
 	)
 	(segment
+		(start 103.148 86.588)
+		(end 95.248 86.588)
+		(width 0.8)
+		(layer "F.Cu")
+		(net "+3.3V")
+	)
+	(segment
 		(start 115.817 72.268)
 		(end 115.817 73.9795)
@@
 		(net "+3.3V")
 	)
+	(via
+		(at 95.248 86.588)
+		(size 1)
+		(drill 0.5)
+		(layers "F.Cu" "B.Cu")
+		(capping no)
+		(covering
+			(front no)
+			(back no)
+		)
+		(plugging
+			(front no)
+			(back no)
+		)
+		(filling no)
+		(net "+3.3V")
+	)
+	(segment
+		(start 95.248 83.659)
+		(end 95.248 86.588)
+		(width 0.8)
+		(layer "B.Cu")
+		(net "+3.3V")
+	)
 	(segment
 		(start 103.648 82.663)
@@
 		(net "/PRG_UART_TX")
 	)
+	(zone
+		(net "GND")
+		(layer "In1.Cu")
+		(name "GNDplane1")
+		(hatch edge 0.5)
+		(priority 1)
+		(connect_pads
+			(clearance 0.5)
+		)
+		(min_thickness 0.25)
+		(fill yes
+			(thermal_gap 0.5)
+			(thermal_bridge_width 0.5)
+			(island_removal_mode 0)
+		)
+		(polygon
+			(pts
+				(xy 77.898 87.554) (xy 77.898 37.554) (xy 127.898 37.554) (xy 127.898 87.554)
+			)
+		)
+	)
+	(zone
+		(net "GND")
+		(layer "In2.Cu")
+		(name "GNDplane2")
+		(hatch edge 0.5)
+		(connect_pads
+			(clearance 0.5)
+		)
+		(min_thickness 0.25)
+		(fill yes
+			(thermal_gap 0.5)
+			(thermal_bridge_width 0.5)
+			(island_removal_mode 0)
+		)
+		(polygon
+			(pts
+				(xy 77.898 87.554) (xy 77.898 37.554) (xy 127.898 37.554) (xy 127.898 87.554)
+			)
+		)
+	)
 	(group ""
