File: neptune-camera-esp/neptune-camera-esp.kicad_pcb (KiCad board)
At the start: 4 copper layers, 50 x 50 mm, 44 parts, among them J1 Conn_02x10_Odd_Even, J2 Conn_02x10_Odd_Even, J3 ov5640, J5 Programmersocket, SW1 EN_Button, SW2 BOOT_Button, U1 ESP32-S3-WROOM-1, U2 TLV74315, U3 TLV74328, U4 AP2112K-3.3, U5 AP2112K-3.3

Commit message: Stiching vias
RJAF
Routing:
- net GND: vias 36 -> 115

Commit message: final
Parts:
- moved R5 2.90 mm to (109.2, 51.8), turned to 0 degrees
- moved R6 1.64 mm to (109.2, 53.1), turned to 180 degrees
Connections:
- U1 pad 11: unconnected-(U1-IO18-Pad11) -> /OV5640_SDA
- U1 pad 12: unconnected-(U1-IO8-Pad12) -> /OV5640_SCL
- U1 pad 15: /OV5640_SDA -> unconnected-(U1-IO3-Pad15)
- U1 pad 16: /OV5640_SCL -> unconnected-(U1-IO46-Pad16)
- U1 pad 26: /D6 -> unconnected-(U1-IO45-Pad26)
- U1 pad 31: /D2 -> /D6
- U1 pad 32: /D5 -> /D2
- U1 pad 33: /D3 -> /D5
- U1 pad 34: /D4 -> /D3
- U1 pad 35: unconnected-(U1-IO42-Pad35) -> /D4
Routing:
- net /D6: track 26.3 -> 35.4 mm
- net /OV5640_SDA: track 27.2 -> 36.0 mm
- net /OV5640_SCL: track 27.1 -> 34.8 mm
- net +3.3VA: track 68.7 -> 65.6 mm
- net /D4: track 39.8 -> 41.0 mm
- net /D3: track 38.4 -> 39.6 mm
- net /D5: track 37.0 -> 38.2 mm
- net /D2: track 35.6 -> 36.8 mm
- net GND: vias 115 -> 108

Commit message: prod
Parts:
- added C27: NEFORRASZDBE_DEBUG_22PF, Capacitor_SMD:C_0402_1005Metric, B.Cu at (95.6, 65.6)
Routing:
- net GND: track 108.6 -> 109.7 mm
- net /PCLK: track 26.0 -> 27.1 mm
Other:
- board text added: "revision 2.0-ESP Project Neptune"
- board text removed: "revision 1.1 Project Neptune"

Commit message: sd card added
Parts:
- added C28: 1uF, Capacitor_SMD:C_0603_1608Metric, F.Cu at (93.8, 39.9)
- added C29: 100nF, Capacitor_SMD:C_0402_1005Metric, F.Cu at (95.1, 40.2)
- added J4: Micro_SD_Card_Det2, Connector_Card:microSD_HC_Hirose_DM3D-SF, F.Cu at (101.3, 47.9)
- added R10: 10k, Resistor_SMD:R_0402_1005Metric, F.Cu at (111.8, 48.0)
- added R11: 10k, Resistor_SMD:R_0402_1005Metric, F.Cu at (111.8, 45.5)
- added R7: 10k, Resistor_SMD:R_0402_1005Metric, F.Cu at (111.8, 44.2)
- added R8: 10k, Resistor_SMD:R_0402_1005Metric, F.Cu at (111.8, 42.9)
- added R9: 10k, Resistor_SMD:R_0402_1005Metric, F.Cu at (111.8, 41.7)
- moved R2 5.70 mm to (107.8, 59.5), turned to 0 degrees
- moved C21 3.01 mm to (107.8, 58.0), turned to 0 degrees
- moved R1 3.00 mm to (107.9, 56.9), turned to 0 degrees
Connections:
- U1 pad 6: unconnected-(U1-IO6-Pad6) -> /SD_DAT0
- U1 pad 7: unconnected-(U1-IO7-Pad7) -> /SD_CLK
- U1 pad 8: unconnected-(U1-IO15-Pad8) -> /SD_CMD
Routing:
- net Net-(J4-DAT2): track 0.00 -> 15.2 mm, vias 0 -> 2
- net /SD_CMD: track 0.00 -> 15.1 mm, vias 0 -> 1
- net Net-(J4-DAT3/CD): track 0.00 -> 13.6 mm, vias 0 -> 2
- net +3.3VA: track 65.6 -> 79.0 mm
- net GND: track 109.7 -> 96.9 mm, vias 108 -> 97
- net /SD_CLK: track 0.00 -> 11.5 mm, vias 0 -> 1
- net /SD_DAT0: track 0.00 -> 9.61 mm, vias 0 -> 1
- net Net-(J4-DAT1): track 0.00 -> 7.28 mm
- net /CAM_RESET: track 26.4 -> 31.1 mm
- net /EN: track 27.8 -> 30.0 mm
- net /PRG_UART_RX: track 28.5 -> 29.6 mm
- net /PRG_UART_TX: track 28.4 -> 29.0 mm
- net /CAM_PWDN: track 27.8 -> 28.3 mm
Other:
- board text added: "revision 2.1 Project Neptune"
- board text removed: "revision 2.0-ESP Project Neptune"

Commit message: Stiching
RJAF
Routing:
- net GND: vias 97 -> 101

Commit message: SDC slot
RKJAF
Connections:
- J4 pad 10: GND -> unconnected-(J4-DET_A-Pad10)
- J4 pad 9: GND -> unconnected-(J4-DET_B-Pad9)
Routing:
- net GND: track 96.9 -> 95.1 mm, vias 101 -> 99
Changed lines of the file:
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@@
 			(size 1.45 1)
 			(layers "F.Cu" "F.Mask" "F.Paste")
-			(net "GND")
+			(net "unconnected-(J4-DET_B-Pad9)")
 			(pinfunction "DET_B_9")
-			(pintype "passive")
+			(pintype "passive+no_connect")
 		)
 		(pad "10" smd rect
@@
 			(size 1 1.55)
 			(layers "F.Cu" "F.Mask" "F.Paste")
-			(net "GND")
+			(net "unconnected-(J4-DET_A-Pad10)")
 			(pinfunction "DET_A_10")
-			(pintype "passive")
+			(pintype "passive+no_connect")
 		)
 		(pad "SH" smd rect
@@
 	)
 	(segment
-		(start 95.703 53.376)
-		(end 96.603 53.376)
-		(width 0.5)
-		(layer "F.Cu")
-		(net "GND")
-	)
-	(segment
 		(start 114.267 77.0795)
 		(end 114.267 75.5295)
@@
 	)
 	(segment
-		(start 106.928 51.801)
-		(end 106.928 52.701)
-		(width 0.5)
-		(layer "F.Cu")
-		(net "GND")
-	)
-	(segment
 		(start 81.999 48.0245)
 		(end 81.999 50.046)
@@
 	)
 	(via
-		(at 96.603 53.376)
-		(size 0.6)
-		(drill 0.3)
-		(layers "F.Cu" "B.Cu")
-		(net "GND")
-	)
-	(via
 		(at 106.439 50.301)
 		(size 0.8)
@@
 		(net "GND")
 	)
-	(via
-		(at 106.928 52.701)
-		(size 0.6)
-		(drill 0.3)
-		(layers "F.Cu" "B.Cu")
-		(net "GND")
-	)
