File: neptune-camera-esp/neptune-camera-esp.kicad_sch (KiCad schematic)
At the start: 25 parts, among them J1 Conn_02x10_Odd_Even, J2 Conn_02x10_Odd_Even, J4 Programmersocket, SW1 EN_Button, SW2 BOOT_Button, U1 ESP32-S3-WROOM-1, U2 TLV74315, U3 TLV74328, U4 AP2112K-3.3

Commit message: -
Parts:
- removed J4: Programmersocket, symbol Connector:Conn_01x04_Socket
- added J5: Programmersocket, neptune-camera-esp-footprints:PinSocket_1x05_P2.54mm_Horizontal, symbol Connector:Conn_01x05_Socket
- added R5, R6: 10k, Resistor_SMD:R_0402_1005Metric, symbol Device:R_Small
Connections:
- net +3.3V: now also R5.2, R6.1
- net D2: now also U1.18 (IO10)
- net D3: now also U1.16 (IO46)
- net D4: now also U1.15 (IO3)
- net D5: now also U1.17 (IO9)
- net D6: now also U1.19 (IO11)
- net D7: now also U1.21 (IO13)
- net D8: now also U1.22 (IO14)
- net D9: now also U1.23 (IO21)
- net GND: now also J5.4 (Pin_4), J5.5 (Pin_5)
- net I2C_OBC_SDA: now also U1.7 (IO7); no longer J1.3 (Pin_3)
- net OV5640_SCL: now also U1.31 (IO38), R6.2
- net OV5640_SDA: now also U1.32 (IO39), R5.1
- net PCLK: now also U1.20 (IO12)
- net PRG_UART_RX: now also J5.3 (Pin_3)
- net PRG_UART_TX: now also J5.2 (Pin_2)
- net VCC: now also J5.1 (Pin_1)
- net VSYNC: now also U1.25 (IO48)
- net HSYNC: now reaches U1.24 (IO47)
- net I2C_OBC_SCL: now reaches U1.8 (IO15)
- net I2C_OBC_SCL: now also J1.3 (Pin_3)

Commit message: Production
Connections:
- net LTE_PWRKEY: now also U1.34 (IO41)
- net LTE_RESET: now also U1.35 (IO42)
Changed lines of the file:
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@@
+		)
+	)
+	(label "LTE_RESET"
+		(at 78.74 83.82 0)
+		(effects
+			(font
+				(size 1.27 1.27)
+			)
+			(justify left bottom)
+		)
+	)
+	(label "LTE_PWRKEY"
+		(at 78.74 81.28 0)
+		(effects
+			(font
+				(size 1.27 1.27)
+			)
+			(justify left bottom)
 		)
 	)
