File: neptune-camera-esp/camera.kicad_sch (KiCad schematic)
At the start: 16 parts, among them J3 ov5640, Y1 ECS-2520MVQ-240-BS-TR

Commit message: megyek ebédelni :)
Parts:
- removed C20: 22pF, Capacitor_SMD:C_0402_1005Metric, symbol Device:C_Small
- removed Y1: ECS-2520MVQ-240-BS-TR, neptune-camera-esp-footprints:ECS2520MVQ240BSTR, symbol neptune-camera-esp-symbols:ECS-2520MVQ-240-BS-TR

Commit message: finom volt az ebéd, megyek haza
Changed lines of the file:
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@@
 	(wire
 		(pts
-			(xy 50.8 57.15) (xy 63.5 57.15)
+			(xy 50.8 57.15) (xy 52.07 57.15)
 		)
 		(stroke
@@
 			(width 0)
 			(type default)
-		)
-	)
-	(label "CameraPWDN"
-		(at 62.23 44.45 0)
-		(effects
-			(font
-				(size 1.27 1.27)
-			)
-			(justify left bottom)
-		)
-	)
-	(label "XCLK"
-		(at 63.5 57.15 0)
-		(effects
-			(font
-				(size 1.27 1.27)
-			)
-			(justify left bottom)
-		)
-	)
-	(label "CameraPWDN"
-		(at 158.75 48.26 180)
-		(effects
-			(font
-				(size 1.27 1.27)
-			)
-			(justify right bottom)
-		)
-	)
-	(label "CameraReset"
-		(at 158.75 26.67 180)
-		(effects
-			(font
-				(size 1.27 1.27)
-			)
-			(justify right bottom)
-		)
-	)
-	(label "CameraReset"
-		(at 62.23 39.37 0)
-		(effects
-			(font
-				(size 1.27 1.27)
-			)
-			(justify left bottom)
 		)
 	)
@@
 		)
 	)
+	(hierarchical_label "XCLK"
+		(shape input)
+		(at 52.07 57.15 0)
+		(effects
+			(font
+				(size 1.27 1.27)
+			)
+			(justify left)
+		)
+	)
 	(hierarchical_label "D2"
 		(shape output)
@@
 			)
 			(justify left)
+		)
+	)
+	(hierarchical_label "CameraReset"
+		(shape input)
+		(at 158.75 26.67 180)
+		(effects
+			(font
+				(size 1.27 1.27)
+			)
+			(justify right)
 		)
 	)
@@
 		)
 	)
+	(hierarchical_label "CameraPWDN"
+		(shape input)
+		(at 158.75 48.26 180)
+		(effects
+			(font
+				(size 1.27 1.27)
+			)
+			(justify right)
+		)
+	)
 	(hierarchical_label "D4"
 		(shape output)
@@
 		)
 	)
+	(hierarchical_label "CameraPWDN"
+		(shape input)
+		(at 62.23 44.45 0)
+		(effects
+			(font
+				(size 1.27 1.27)
+			)
+			(justify left)
+		)
+	)
 	(hierarchical_label "D3"
 		(shape output)
@@
 		(effects
 			(font
+				(size 1.27 1.27)
+			)
+			(justify left)
+		)
+	)
+	(hierarchical_label "CameraReset"
+		(shape input)
+		(at 62.23 39.37 0)
+		(effects
+			(font

Commit message: még kellenek stiching viák, meg át kell nézni
Connections:
- net +3.3V: no longer R1.2
- new net +3.3VA: R1.2

Commit message: prod
Parts:
- added C27: NEFORRASZDBE_DEBUG_22PF, Capacitor_SMD:C_0402_1005Metric, symbol Device:C_Small
Connections:
- net GND: now also C27.1
- net PCLK: now also C27.2
Changed lines of the file:
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@@
+	)
+	(junction
+		(at 67.31 67.31)
+		(diameter 0)
+		(color 0 0 0 0)
 	)
 	(junction
@@
 	(wire
 		(pts
+			(xy 67.31 67.31) (xy 74.93 67.31)
+		)
+		(stroke
+			(width 0)
+			(type default)
+		)
+	)
+	(wire
+		(pts
 			(xy 50.8 62.23) (xy 52.07 62.23)
 		)
@@
 	(wire
 		(pts
-			(xy 50.8 67.31) (xy 52.07 67.31)
+			(xy 50.8 67.31) (xy 67.31 67.31)
 		)
 		(stroke
@@
 	(hierarchical_label "PCLK"
 		(shape output)
-		(at 52.07 67.31 0)
+		(at 74.93 67.31 0)
 		(effects
 			(font
@@
 	(symbol
 		(lib_id "power:GND")
+		(at 67.31 72.39 0)
+		(unit 1)
+		(body_style 1)
+		(exclude_from_sim no)
+		(in_bom yes)
+		(on_board yes)
+		(in_pos_files yes)
+		(dnp no)
+		(fields_autoplaced yes)
+		(property "Reference" "#PWR048"
+			(at 67.31 78.74 0)
+			(hide yes)
+			(show_name no)
+			(do_not_autoplace no)
+			(effects
+				(font
+					(size 1.27 1.27)
+				)
+			)
+		)
+		(property "Value" "GND"
+			(at 67.31 77.47 0)
+			(show_name no)
+			(do_not_autoplace no)
+			(effects
+				(font
+					(size 1.27 1.27)
+				)
+			)
+		)
+		(property "Footprint" ""
+			(at 67.31 72.39 0)
+			(hide yes)
+			(show_name no)
+			(do_not_autoplace no)
+			(effects
+				(font
+					(size 1.27 1.27)
+				)
+			)
+		)
+		(property "Datasheet" ""
+			(at 67.31 72.39 0)
+			(hide yes)
+			(show_name no)
+			(do_not_autoplace no)
+			(effects
+				(font
+					(size 1.27 1.27)
+				)
+			)
+		)
+		(property "Description" "Power symbol creates a global label with name \"GND\" , ground"
+			(at 67.31 72.39 0)
+			(hide yes)
+			(show_name no)
+			(do_not_autoplace no)
+			(effects
+				(font
+					(size 1.27 1.27)
+				)
+			)
+		)
+		(pin "1"
+		)
+		(instances
+			(project "neptune-camera-esp"
+				(path "/21f72d0d-5890-47b1-bb90-d92ee48f04f5/0926fe47-5ef5-46ea-8672-59359ad1ad72"
+					(reference "#PWR048")
+					(unit 1)
+				)
+			)
+		)
+	)
+	(symbol
+		(lib_id "power:GND")
 		(at 167.64 48.26 90)
 		(unit 1)
@@
 					(unit 1)
 				)
+			)
+		)
+	)
+	(symbol
+		(lib_id "Device:C_Small")
+		(at 67.31 69.85 180)
+		(unit 1)
+		(body_style 1)
+		(exclude_from_sim no)
+		(in_bom yes)
+		(on_board yes)
+		(in_pos_files yes)
+		(dnp no)
+		(fields_autoplaced yes)
+		(property "Reference" "C27"
+			(at 64.77 71.1138 0)
+			(show_name no)
+			(do_not_autoplace no)
+			(effects
+				(font
+					(size 1.27 1.27)
+				)
+				(justify left)
+			)
+		)
+		(property "Value" "NEFORRASZDBE_DEBUG_22PF"
+			(at 64.77 68.5738 0)
+			(show_name no)
+			(do_not_autoplace no)
+			(effects
+				(font
+					(size 1.27 1.27)
+				)
+				(justify left)
+			)
+		)
+		(property "Footprint" "Capacitor_SMD:C_0402_1005Metric"
+			(at 67.31 69.85 0)
+			(hide yes)
+			(show_name no)
+			(do_not_autoplace no)
+			(effects
+				(font
+					(size 1.27 1.27)
+				)
+			)
+		)
+		(property "Datasheet" ""
+			(at 67.31 69.85 0)
+			(hide yes)
+			(show_name no)
+			(do_not_autoplace no)
+			(effects
+				(font
+					(size 1.27 1.27)
+				)
+			)
+		)
+		(property "Description" "Unpolarized capacitor, small symbol"
+			(at 67.31 69.85 0)
+			(hide yes)
+			(show_name no)
+			(do_not_autoplace no)
+			(effects
+				(font
+					(size 1.27 1.27)
+				)
+			)
+		)
+		(pin "1"
+		)
+		(pin "2"
+		)
+		(instances
+			(project "neptune-camera-esp"
+				(path "/21f72d0d-5890-47b1-bb90-d92ee48f04f5/0926fe47-5ef5-46ea-8672-59359ad1ad72"
+					(reference "C27")
+					(unit 1)
+				)

Commit message: sd card added
Changed lines of the file:
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@@
 		(in_pos_files yes)
 		(dnp no)
-		(fields_autoplaced yes)
 		(property "Reference" "C27"
-			(at 64.77 71.1138 0)
+			(at 69.596 69.596 0)
 			(show_name no)
 			(do_not_autoplace no)
@@
 					(size 1.27 1.27)
 				)
-				(justify left)
+				(justify right)
 			)
 		)
 		(property "Value" "NEFORRASZDBE_DEBUG_22PF"
-			(at 64.77 68.5738 0)
+			(at 69.596 72.136 0)
 			(show_name no)
 			(do_not_autoplace no)
@@
 					(size 1.27 1.27)
 				)
-				(justify left)
+				(justify right)
 			)
 		)
